Commit message: attached_a_leg_not_right_pos

File: drake_sim/urdf/quadruped_base.urdf (robot description, URDF)
Before this commit: robot quadruped_base, 2 links, 0 joints
Links:
- removed link quadruped_base
- added link main_body, mass 6.7053012; collision mesh filename=meshes/body_collision.obj; visual mesh filename=meshes/body.obj
