Commit message: body_collisions

File: drake_sim/urdf/ntnu_legFL.urdf (robot description, URDF)
Before this commit: robot ntnu_leg, 5 links, 4 joints
Links:
- link MH: geometry collision mesh filename=meshes/MH_collisionSW.obj; visual mesh filename=meshes/MH.obj
- link link11: geometry collision mesh filename=meshes/link11_collisionSW.obj; visual mesh filename=meshes/link11.obj
- link link12: geometry collision mesh filename=meshes/link12_collisionSW.obj; visual mesh filename=meshes/link12.obj
- link link21: geometry collision mesh filename=meshes/link21_collisionSW.obj; visual mesh filename=meshes/link21.obj
- link link22: geometry collision mesh filename=meshes/link22_collisionSW.obj; visual mesh filename=meshes/link22.obj

File: drake_sim/urdf/ntnu_legFR.urdf (robot description, URDF)
Before this commit: robot ntnu_leg, 5 links, 4 joints
Links:
- link MH: geometry collision mesh filename=meshes/MH_collisionSW.obj; visual mesh filename=meshes/MH.obj
- link link11: geometry collision mesh filename=meshes/link11_collisionSW.obj; visual mesh filename=meshes/link11.obj
- link link12: geometry collision mesh filename=meshes/link12_collisionSW.obj; visual mesh filename=meshes/link12.obj
- link link21: geometry collision mesh filename=meshes/link21_collisionSW.obj; visual mesh filename=meshes/link21.obj
- link link22: geometry collision mesh filename=meshes/link22_collisionSW.obj; visual mesh filename=meshes/link22.obj

File: drake_sim/urdf/ntnu_legRL.urdf (robot description, URDF)
Before this commit: robot ntnu_leg, 5 links, 4 joints
Links:
- link MH: geometry collision mesh filename=meshes/MH_collisionSW.obj; visual mesh filename=meshes/MH.obj
- link link11: geometry collision mesh filename=meshes/link11_collisionSW.obj; visual mesh filename=meshes/link11.obj
- link link12: geometry collision mesh filename=meshes/link12_collisionSW.obj; visual mesh filename=meshes/link12.obj
- link link21: geometry collision mesh filename=meshes/link21_collisionSW.obj; visual mesh filename=meshes/link21.obj
- link link22: geometry collision mesh filename=meshes/link22_collisionSW.obj; visual mesh filename=meshes/link22.obj

File: drake_sim/urdf/quadruped_base.urdf (robot description, URDF)
Before this commit: robot quadruped_base, 2 links, 0 joints
Links:
- link main_body: geometry collision mesh filename=meshes/body_MH_front_cover.obj; collision mesh filename=meshes/body_MH_front_motors.obj
